Commit message: aruco cube add

File: src/shesnar/urdf/lidar.xacro (robot description, xacro)
@@ -26,5 +26,5 @@
         <parent link="body"/>
         <child link="laser_frame"/>
-        <origin xyz="0 0 0.41" rpy="0 0 -2.085"/>
+        <origin xyz="0 0 0.338" rpy="0 0 -1.57"/>
     </joint>
     <link name="laser_frame">
@@ -43,8 +43,8 @@
         </xacro:inertial_cylinder>
     </link>
-    <link name="aruco">
+    <link name="top_aruco">
         <visual>
             <geometry>
-                 <mesh filename="file://$(find shesnar)/meshes/aruco_plane.obj" scale="0.5 0.5 0.5"/>
+                 <mesh filename="file://$(find shesnar)/meshes/aruco_plane-7.obj" scale="0.5 0.5 0.5"/>
             </geometry>
         </visual>
@@ -52,6 +52,54 @@
     <joint name="aruco_joint" type="fixed">
         <parent link="laser_frame"/>
-        <child link="aruco"/>
-        <origin xyz="0 0 0.0225" rpy="1.571 0 2.085"/>
+        <child link="top_aruco"/>
+        <origin xyz="0 0 0.0935" rpy="1.571 0 1.57"/>
+    </joint>
+    <link name="right_aruco">
+        <visual>
+            <geometry>
+                 <mesh filename="file://$(find shesnar)/meshes/aruco_plane-77.obj" scale="0.5 0.5 0.5"/>
+            </geometry>
+        </visual>
+    </link>
+    <joint name="right_aruco_joint" type="fixed">
+        <parent link="top_aruco"/>
+        <child link="right_aruco"/>
+        <origin xyz="0 -0.0415 0.048" rpy="1.571 0 0"/>
+    </joint>
+    <link name="left_aruco">
+        <visual>
+            <geometry>
+                 <mesh filename="file://$(find shesnar)/meshes/aruco_plane-78.obj" scale="0.5 0.5 0.5"/>
+            </geometry>
+        </visual>
+    </link>
+    <joint name="left_aruco_joint" type="fixed">
+        <parent link="top_aruco"/>
+        <child link="left_aruco"/>
+        <origin xyz="0 -0.0415 -0.048" rpy="-1.571 0 0"/>
+    </joint>
+    <link name="back_aruco">
+        <visual>
+            <geometry>
+                 <mesh filename="file://$(find shesnar)/meshes/aruco_plane-83.obj" scale="0.5 0.5 0.5"/>
+            </geometry>
+        </visual>
+    </link>
+    <joint name="back_aruco_joint" type="fixed">
+        <parent link="top_aruco"/>
+        <child link="back_aruco"/>
+        <origin xyz="-0.048 -0.0415 0" rpy="0 0 1.571"/>
+    </joint>
+    <link name="forward_aruco">
+        <visual>
+            <geometry>
+                 <mesh filename="file://$(find shesnar)/meshes/aruco_plane-88.obj" scale="0.5 0.5 0.5"/>
+            </geometry>
+        </visual>
+    </link>
+    <joint name="forward_aruco_joint" type="fixed">
+        <parent link="top_aruco"/>
+        <child link="forward_aruco"/>
+        <origin xyz="0.048 -0.0415 0" rpy="0 0 -1.571"/>
     </joint>
 </robot>

Commit message: added info reading from side markers

File: src/shesnar/urdf/lidar.xacro (robot description, xacro)
@@ -77,5 +77,5 @@
         <parent link="top_aruco"/>
         <child link="left_aruco"/>
-        <origin xyz="0 -0.0415 -0.048" rpy="-1.571 0 0"/>
+        <origin xyz="0 -0.0415 -0.048" rpy="-1.571 0 -3.14"/>
     </joint>
     <link name="back_aruco">
@@ -89,5 +89,5 @@
         <parent link="top_aruco"/>
         <child link="back_aruco"/>
-        <origin xyz="-0.048 -0.0415 0" rpy="0 0 1.571"/>
+        <origin xyz="-0.048 -0.0415 0" rpy="0 -1.571 1.571"/>
     </joint>
     <link name="forward_aruco">
@@ -101,5 +101,5 @@
         <parent link="top_aruco"/>
         <child link="forward_aruco"/>
-        <origin xyz="0.048 -0.0415 0" rpy="0 0 -1.571"/>
+        <origin xyz="0.048 -0.0415 0" rpy="0 1.571 -1.571"/>
     </joint>
 </robot>

Commit message: fixed sizes and places of robot aruco

File: src/shesnar/urdf/lidar.xacro (robot description, xacro)
@@ -43,8 +43,23 @@
         </xacro:inertial_cylinder>
     </link>
+    <!-- ARUCO - МАРКЕРЫ -->
+    <!-- высота верхнего маркера относительно звена лидара // P.S.: до этого было 0.0935 -->
+    <xacro:property name="top_marker_height" value="0.102" />
+    <!-- масштабирование верхнего маркера -->
+    <!-- оригинальный размер маркера в модели - 0.2 м (с белыми краями); реальный на роботе - 0.07 м (без учёта белого края), 0.0933 м (с учётом) -->
+    <!-- (0.07 / 6 * 8) / 0.2 = 0.466666667 -->
+    <xacro:property name="top_marker_scale" value="0.466666667" />
+    <!--отступ в горизонтальной плоскости (вперёд/назад/вбок)-->
+    <xacro:property name="side_marker_horizontal_offset" value="0.048" />
+    <!-- отступ вниз по высоте относительно плоскости верхнего марекра // P.S.: до этого было -0.0415-->
+    <xacro:property name="side_marker_vertical_offset" value="-0.07" />
+    <!-- масштабирование боковых маркеров -->
+    <!-- оригинальный размер маркеров в модели - 0.2 м (с белыми краями); реальные на роботе - 0.06 м (без учёта белого края), 0.08 м (с учётом) -->
+    <!-- (0.06 / 6 * 8) / 0.2 = 0.4 -->
+    <xacro:property name="side_marker_scale" value="0.4" />
     <link name="top_aruco">
         <visual>
             <geometry>
-                 <mesh filename="file://$(find shesnar)/meshes/aruco_plane-7.obj" scale="0.5 0.5 0.5"/>
+                 <mesh filename="file://$(find shesnar)/meshes/aruco_plane-7.obj" scale="${top_marker_scale} 0.005 ${top_marker_scale}"/>
             </geometry>
         </visual>
@@ -53,10 +68,10 @@
         <parent link="laser_frame"/>
         <child link="top_aruco"/>
-        <origin xyz="0 0 0.0935" rpy="1.571 0 1.57"/>
+        <origin xyz="0 0 ${top_marker_height}" rpy="1.571 0 1.571"/>
     </joint>
     <link name="right_aruco">
         <visual>
             <geometry>
-                 <mesh filename="file://$(find shesnar)/meshes/aruco_plane-77.obj" scale="0.5 0.5 0.5"/>
+                 <mesh filename="file://$(find shesnar)/meshes/aruco_plane-77.obj" scale="${side_marker_scale} 0.005 ${side_marker_scale}"/>
             </geometry>
         </visual>
@@ -65,10 +80,10 @@
         <parent link="top_aruco"/>
         <child link="right_aruco"/>
-        <origin xyz="0 -0.0415 0.048" rpy="1.571 0 0"/>
+        <origin xyz="0 ${side_marker_vertical_offset} ${side_marker_horizontal_offset}" rpy="1.571 0 0"/>
     </joint>
     <link name="left_aruco">
         <visual>
             <geometry>
-                 <mesh filename="file://$(find shesnar)/meshes/aruco_plane-78.obj" scale="0.5 0.5 0.5"/>
+                 <mesh filename="file://$(find shesnar)/meshes/aruco_plane-78.obj" scale="${side_marker_scale} 0.005 ${side_marker_scale}"/>
             </geometry>
         </visual>
@@ -77,10 +92,10 @@
         <parent link="top_aruco"/>
         <child link="left_aruco"/>
-        <origin xyz="0 -0.0415 -0.048" rpy="-1.571 0 -3.14"/>
+        <origin xyz="0 ${side_marker_vertical_offset} ${-side_marker_horizontal_offset}" rpy="-1.571 0 -3.14"/>
     </joint>
     <link name="back_aruco">
         <visual>
             <geometry>
-                 <mesh filename="file://$(find shesnar)/meshes/aruco_plane-83.obj" scale="0.5 0.5 0.5"/>
+                 <mesh filename="file://$(find shesnar)/meshes/aruco_plane-83.obj" scale="${side_marker_scale} 0.005 ${side_marker_scale}"/>
             </geometry>
         </visual>
@@ -89,10 +104,10 @@
         <parent link="top_aruco"/>
         <child link="back_aruco"/>
-        <origin xyz="-0.048 -0.0415 0" rpy="0 -1.571 1.571"/>
+        <origin xyz="${-side_marker_horizontal_offset} ${side_marker_vertical_offset} 0" rpy="0 -1.571 1.571"/>
     </joint>
     <link name="forward_aruco">
         <visual>
             <geometry>
-                 <mesh filename="file://$(find shesnar)/meshes/aruco_plane-88.obj" scale="0.5 0.5 0.5"/>
+                 <mesh filename="file://$(find shesnar)/meshes/aruco_plane-88.obj" scale="${side_marker_scale} 0.005 ${side_marker_scale}"/>
             </geometry>
         </visual>
@@ -101,5 +116,5 @@
         <parent link="top_aruco"/>
         <child link="forward_aruco"/>
-        <origin xyz="0.048 -0.0415 0" rpy="0 1.571 -1.571"/>
+        <origin xyz="${side_marker_horizontal_offset} ${side_marker_vertical_offset} 0" rpy="0 1.571 -1.571"/>
     </joint>
 </robot>
